Commit message: Added the version to the xacros.

File: duatic_dynaarm_driver/duatic_dynaarm_driver/urdf/dynaarm.ros2control.xacro (robot description, xacro)
@@ -62,5 +62,13 @@
     </joint>
   </xacro:macro>
-  <xacro:macro name="dynaarm_ros2_control" params="tf_prefix namespace:='' ethercat_bus start_in_freeze_mode drive_parameter_folder:='' ethercat_addresses mode">
+  <xacro:macro name="dynaarm_ros2_control"
+               params="tf_prefix
+                       namespace:=''
+                       ethercat_bus
+                       start_in_freeze_mode
+                       drive_parameter_folder:=''
+                       version
+                       ethercat_addresses
+                       mode">
     <!--Allow the user to pass a custom folder for drive parameters-->
     <xacro:property name="default_drive_parameter_folder" value="$(find duatic_dynaarm_driver)/config/${version}" />

File: duatic_dynaarm_driver/duatic_dynaarm_driver/urdf/dynaarm.urdf.xacro (robot description, xacro)
@@ -24,5 +24,16 @@
 <robot name="dynaarm" xmlns:xacro="http://www.ros.org/wiki/xacro">
     <xacro:macro name="dynaarm"
-    params="tf_prefix parent_link collision:='simple' dof mode ethercat_bus drive_order:='' start_in_freeze_mode:=false drive_parameter_folder:='' covers version *origin">
+                 params="tf_prefix
+                         parent_link
+                         collision:='simple'
+                         dof
+                         mode
+                         ethercat_bus
+                         drive_order:=''
+                         start_in_freeze_mode:=false
+                         drive_parameter_folder:=''
+                         covers
+                         version
+                         *origin">
         <xacro:include filename="$(find duatic_dynaarm_description)/urdf/dynaarm.urdf.xacro" />
         <xacro:include filename="$(find duatic_dynaarm_driver)/urdf/dynaarm.ros2control.xacro" />
@@ -42,5 +53,5 @@
             <xacro:insert_block name="origin" />
         </xacro:dynaarm_description>
-        <!-- Creatte the ros2control part-->
+        <!-- Create the ros2control part-->
         <xacro:dynaarm_ros2_control tf_prefix="${tf_prefix}"
                                     ethercat_bus="${ethercat_bus}"
@@ -48,4 +59,5 @@
                                     drive_parameter_folder="${drive_parameter_folder}"
                                     ethercat_addresses="${ethercat_addresses}"
+                                    version="${version}"
                                     mode="${mode}"/>
     </xacro:macro>
