Commit message: rework to new urdf structure

File: duatic_dynaarm_driver/urdf/dynaarm.ros2control.xacro (robot description, xacro)
@@ -22,45 +22,74 @@
 -->
 <robot xmlns:xacro="http://www.ros.org/wiki/xacro">
-  <xacro:macro name="dynaarm_joint_ros2control_joint_interfaces">
-    <state_interface name="position">
-        <!-- Slightly offset the initial position for the gazebo sim-->
-        <param name="initial_value">0.05</param>
-    </state_interface>
-    <state_interface name="velocity" />
-    <state_interface name="effort" />
-    <state_interface name="acceleration" />
-    <state_interface name="position_commanded" />
-    <state_interface name="velocity_commanded" />
-    <state_interface name="acceleration_commanded" />
-    <state_interface name="effort_commanded" />
-    <state_interface name="temperature_system" />
-    <state_interface name="temperature_coil_A" />
-    <state_interface name="temperature_coil_B" />
-    <state_interface name="temperature_coil_C" />
-    <state_interface name="bus_voltage" />
-    <command_interface name="position" />
-    <command_interface name="velocity" />
-    <command_interface name="effort" />
-    <command_interface name="p_gain" />
-    <command_interface name="i_gain" />
-    <command_interface name="d_gain" />
-  </xacro:macro>
-  <xacro:macro name="dynaarm_ros2control_joint" params="name address mode">
-    <joint name="${name}">
+  <xacro:include filename="$(find duatic_duadrive_interface)/urdf/duadrive_interface.urdf.xacro" />
+  <!--Macro which only creates the joints of a dynaarm (used for combined hardware interfaces)-->
+  <xacro:macro name="dynaarm_ros2_control_joints"
+      params="
+        ethercat_bus
+        mode
+        parent_unit
+        version
+        tf_prefix">
+      <!--Allow the user to pass a custom folder for drive parameters-->
+      <xacro:property name="default_drive_parameter_folder" value="$(find duatic_dynaarm_driver)/config/${version}" />
+      <xacro:if value="${drive_parameter_folder == ''}">
+        <xacro:property name="drive_parameter_folder_internal" value="${default_drive_parameter_folder}" />
+      </xacro:if>
+      <xacro:unless value="${drive_parameter_folder == ''}">
+        <xacro:property name="drive_parameter_folder_internal" value="${drive_parameter_folder}" />
+      </xacro:unless>
+      <xacro:if value="${dof >= 1}">
+        <xacro:duadrive_interface_joint name="${tf_prefix}shoulder_rotation"
+          ethercat_address="${ethercat_addresses['shoulder_rotation']}"
+          ethercat_bus="${ethercat_bus}"
+          mode="${mode}"
+          parent_unit="${parent_unit}"
+          drive_parameter_file_path="${drive_parameter_folder_internal}/shoulder_rotation.yaml" />
+      </xacro:if>
+      <xacro:if value="${dof >= 2}">
+        <xacro:duadrive_interface_joint name="${tf_prefix}shoulder_flexion"
+          ethercat_address="${ethercat_addresses['shoulder_flexion']}"
+          ethercat_bus="${ethercat_bus}"
+          mode="${mode}"
+          parent_unit="${parent_unit}"
+          drive_parameter_file_path="${drive_parameter_folder_internal}/shoulder_flexion.yaml" />
+      </xacro:if>
+      <xacro:if value="${dof >= 3}">
+        <xacro:duadrive_interface_joint name="${tf_prefix}elbow_flexion"
+          ethercat_address="${ethercat_addresses['elbow_flexion']}"
+          ethercat_bus="${ethercat_bus}"
+          mode="${mode}"
+          parent_unit="${parent_unit}"
+          drive_parameter_file_path="${drive_parameter_folder_internal}/elbow_flexion.yaml" />
+      </xacro:if>
+      <xacro:if value="${dof >= 4}">
+        <xacro:duadrive_interface_joint name="${tf_prefix}forearm_rotation"
+          ethercat_address="${ethercat_addresses['forearm_rotation']}"
+          ethercat_bus="${ethercat_bus}"
+          mode="${mode}"
+          parent_unit="${parent_unit}"
+          drive_parameter_file_path="${drive_parameter_folder_internal}/forearm_rotation.yaml" />
+      </xacro:if>
+      <xacro:if value="${dof >= 5}">
+        <xacro:duadrive_interface_joint name="${tf_prefix}wrist_flexion"
+          ethercat_address="${ethercat_addresses['wrist_flexion']}"
+          ethercat_bus="${ethercat_bus}"
+          mode="${mode}"
+          parent_unit="${parent_unit}"
+          drive_parameter_file_path="${drive_parameter_folder_internal}/wrist_flexion.yaml" />
+      </xacro:if>
+      <xacro:if value="${dof >= 6}">
+        <xacro:duadrive_interface_joint name="${tf_prefix}wrist_rotation"
+          ethercat_address="${ethercat_addresses['wrist_rotation']}"
+          ethercat_bus="${ethercat_bus}"
+          mode="${mode}"
+          parent_unit="${parent_unit}"
+          drive_parameter_file_path="${drive_parameter_folder_internal}/wrist_rotation.yaml" />
+      </xacro:if>
       <xacro:if value="${mode != 'isaac'}">
-        <param name="address">${address}</param>
-        <xacro:dynaarm_joint_ros2control_joint_interfaces />
+        <gpio name="${parent_unit}">
+          <command_interface name="freeze_mode" />
+        </gpio>
       </xacro:if>
-      <xacro:if value="${mode == 'isaac'}">
-        <command_interface name="position" />
-        <command_interface name="velocity" />
-        <command_interface name="effort" />
-        <state_interface name="position">
-          <param name="initial_value">0.0</param>
-        </state_interface>
-        <state_interface name="velocity" />
-        <state_interface name="effort" />
-      </xacro:if>
-    </joint>
   </xacro:macro>
   <xacro:macro name="dynaarm_ros2_control"
@@ -73,15 +102,8 @@
                        ethercat_addresses
                        mode">
-    <!--Allow the user to pass a custom folder for drive parameters-->
-    <xacro:property name="default_drive_parameter_folder" value="$(find duatic_dynaarm_driver)/config/${version}" />
-    <xacro:if value="${drive_parameter_folder == ''}">
-      <xacro:property name="drive_parameter_folder_internal" value="${default_drive_parameter_folder}" />
-    </xacro:if>
-    <xacro:unless value="${drive_parameter_folder == ''}">
-      <xacro:property name="drive_parameter_folder_internal" value="${drive_parameter_folder}" />
-    </xacro:unless>
     <ros2_control name="${tf_prefix}DynaarmSystem" type="system">
       <hardware>
         <xacro:if value="${mode == 'isaac'}">
+          <!--Special case for isaac gym-->
           <plugin>joint_state_topic_hardware_interface/JointStateTopicSystem</plugin>
           <param name="joint_states_topic">isaac_joint_states</param>
@@ -91,47 +113,29 @@
         </xacro:if>
         <xacro:if value="${mode == 'sim'}">
+          <!--Special case for gazebo simulation-->
           <plugin>gz_ros2_control/GazeboSimSystem</plugin>
         </xacro:if>
         <xacro:if value="${mode == 'mock'}">
+          <!--Special case for mocked hardware (simple feedback)-->
           <plugin>duatic::dynaarm_driver/DynaArmHardwareInterfaceMock</plugin>
           <param name="ethercat_bus">${ethercat_bus}</param>
           <param name="tf_prefix">${tf_prefix}</param>
           <param name="start_in_freeze_mode">${start_in_freeze_mode}</param>
-          <param name="drive_parameter_folder">${drive_parameter_folder_internal}</param>
-          <param name="drive_parameter_folder_default">${default_drive_parameter_folder}</param>
           <param name="initial_positions">[0.05, 0.05, 0.10, 0.05, 0.05, 0.05]</param>
         </xacro:if>
         <xacro:if value="${mode == 'real'}">
+          <!--Special case for real hardware-->
           <plugin>duatic::dynaarm_driver/DynaArmHardwareInterfaceReal</plugin>
           <param name="ethercat_bus">${ethercat_bus}</param>
           <param name="tf_prefix">${tf_prefix}</param>
           <param name="start_in_freeze_mode">${start_in_freeze_mode}</param>
-          <param name="drive_parameter_folder">${drive_parameter_folder_internal}</param>
-          <param name="drive_parameter_folder_default">${default_drive_parameter_folder}</param>
         </xacro:if>
       </hardware>
-      <xacro:if value="${dof >= 1}">
-        <xacro:dynaarm_ros2control_joint name="${tf_prefix}shoulder_rotation" address="${ethercat_addresses['shoulder_rotation']}" mode="${mode}" />
-      </xacro:if>
-      <xacro:if value="${dof >= 2}">
-        <xacro:dynaarm_ros2control_joint name="${tf_prefix}shoulder_flexion" address="${ethercat_addresses['shoulder_flexion']}" mode="${mode}" />
-      </xacro:if>
-      <xacro:if value="${dof >= 3}">
-        <xacro:dynaarm_ros2control_joint name="${tf_prefix}elbow_flexion" address="${ethercat_addresses['elbow_flexion']}" mode="${mode}" />
-      </xacro:if>
-      <xacro:if value="${dof >= 4}">
-        <xacro:dynaarm_ros2control_joint name="${tf_prefix}forearm_rotation" address="${ethercat_addresses['forearm_rotation']}" mode="${mode}" />
-      </xacro:if>
-      <xacro:if value="${dof >= 5}">
-        <xacro:dynaarm_ros2control_joint name="${tf_prefix}wrist_flexion" address="${ethercat_addresses['wrist_flexion']}" mode="${mode}" />
-      </xacro:if>
-      <xacro:if value="${dof >= 6}">
-        <xacro:dynaarm_ros2control_joint name="${tf_prefix}wrist_rotation" address="${ethercat_addresses['wrist_rotation']}" mode="${mode}" />
-      </xacro:if>
-      <xacro:if value="${mode != 'isaac'}">
-        <gpio name="${tf_prefix}DynaarmSystem">
-          <command_interface name="freeze_mode" />
-        </gpio>
-      </xacro:if>
+      <xacro:dynaarm_ros2_control_joints
+        tf_prefix="${tf_prefix}"
+        mode="${mode}"
+        version="${version}"
+        ethercat_bus="${ethercat_bus}"
+        parent_unit="${tf_prefix}DynaarmSystem"/>
     </ros2_control>
   </xacro:macro>
